File: Kicad/Solenoid pulser.kicad_pcb (KiCad board)
At the start: 2 copper layers, 33 x 68.6 mm, 26 parts, among them J1 Screw_Terminal_01x02, J2 Screw_Terminal_01x02, J3 Screw_Terminal_01x02, Q1 TIP122, SW1 SW_Push, U1 NE555P

Commit message: Tweak pcb and 3d design.
Parts:
- removed LOGO1: Logo_Open_Hardware_Small, Symbol:OSHW-Symbol_6.7x6mm_Copper
Routing:
- net /trigger: track 53.2 -> 54.2 mm
- net GND: track 112.4 -> 113.5 mm
Other:
- outline, holes or cut-outs redrawn
- board text added: "Solenoid pulser for 12V JF-0530B 2021-09-20 V1.0"
- board text removed: "Solenoid pulser for 12V JF-0530B 2021-08-06 V1.0 https://atoomnet.net/"
