File: Kicad/Solenoid pulser.sch (KiCad schematic (older format))
At the start: 26 parts, among them J1 Screw_Terminal_01x02, J2 Screw_Terminal_01x02, J3 Screw_Terminal_01x02, Q1 TIP122, SW1 SW_Push, U1 NE555P

Commit message: Tweak pcb and 3d design.
Parts:
- removed LOGO1: Logo_Open_Hardware_Small, Symbol:OSHW-Symbol_6.7x6mm_Copper, symbol Graphic:Logo_Open_Hardware_Small
Changed lines of the file:
@@
 Sheet 1 1
 Title ""
-Date ""
+Date "2021-09-20"
 Rev ""
 Comp ""
@@
 	1    0    0    -1
 $EndComp
-$Comp
-L Graphic:Logo_Open_Hardware_Small LOGO1
-U 1 1 6116083E
-P 7250 6850
-F 0 "LOGO1" H 7497 6875 50  0000 L CNN
-F 1 "Logo_Open_Hardware_Small" H 7250 6625 50  0001 C CNN
-F 2 "Symbol:OSHW-Symbol_6.7x6mm_Copper" H 7250 6850 50  0001 C CNN
-F 3 "~" H 7250 6850 50  0001 C CNN
-	1    7250 6850
-	1    0    0    -1
-$EndComp
